File: pace-core/pace-core.kicad_pcb (KiCad board)
At the start: 4 copper layers, 100 x 100 mm, 155 parts, among them CN1 XT90PW-M.G.Y, CN2 SMTSOM330BTR, CN3 SMTSOM330BTR, CN4 SMTSOM330BTR, CN5 SMTSOM330BTR, CN6 SMTSOM330BTR, CN7 SMTSOM330BTR, J1 MotorOut, J2 Wiz5500-Coprocessor-BoB, J3 Conn_01x05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

Commit message: tidy up
Routing:
- net Net-(USB1-CC2): track 6.57 -> 8.59 mm, vias 0 -> 2
