File: pace-core/pace-mechanicals.kicad_sch (KiCad schematic)
At the start: 31 parts, among them CN2 SMTSOM330BTR, CN3 SMTSOM330BTR, CN4 SMTSOM330BTR, CN5 SMTSOM330BTR, CN6 SMTSOM330BTR, CN7 SMTSOM330BTR, J4 Conn_02x05_Odd_Even, SW1 SKRPACE010, SW2 SKRPACE010, U10 LM75ADP,118, U11 LM75ADP,118, U8 LM75ADP,118, U9 LM75ADP,118

Commit message: updated shematic with test point image
Other:
- note removed: "<testpoint_img>"
- moved on the sheet: C31, C32, C33, C34, CN2, CN3, CN4, CN5, CN6, CN7, D1, D2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

Commit message: tidy up
Changed lines of the file:
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@@
 	(wire
 		(pts
-			(xy 39.37 50.8) (xy 46.99 50.8)
+			(xy 38.1 50.8) (xy 46.99 50.8)
 		)
 		(stroke
@@
 	(symbol
 		(lib_id "power:GND")
-		(at 39.37 50.8 0)
+		(at 38.1 50.8 0)
 		(unit 1)
 		(body_style 1)
@@
 		(dnp no)
 		(property "Reference" "#PWR028"
-			(at 39.37 57.15 0)
+			(at 38.1 57.15 0)
 			(hide yes)
 			(show_name no)
@@
 		)
 		(property "Value" "GND"
-			(at 36.83 51.054 0)
+			(at 35.56 51.054 0)
 			(show_name no)
 			(do_not_autoplace no)
@@
 		)
 		(property "Footprint" ""
-			(at 39.37 50.8 0)
+			(at 38.1 50.8 0)
 			(hide yes)
 			(show_name no)
@@
 		)
 		(property "Datasheet" ""
-			(at 39.37 50.8 0)
+			(at 38.1 50.8 0)
 			(hide yes)
 			(show_name no)
@@
 		)
 		(property "Description" "Power symbol creates a global label with name \"GND\" , ground"
-			(at 39.37 50.8 0)
+			(at 38.1 50.8 0)
 			(hide yes)
 			(show_name no)
