File: pace-core/pace-mechanicals.kicad_sch (KiCad schematic)
At the start: 31 parts, among them CN2 SMTSOM330BTR, CN3 SMTSOM330BTR, CN4 SMTSOM330BTR, CN5 SMTSOM330BTR, CN6 SMTSOM330BTR, CN7 SMTSOM330BTR, J4 Conn_02x05_Odd_Even, SW1 SKRPACE010, SW2 SKRPACE010, U10 LM75ADP,118, U11 LM75ADP,118, U8 LM75ADP,118, U9 LM75ADP,118

Commit message: design checkpoint: v1 repackage — new connectors, footprints, and layout updates
- Add JST SH/SR series, XT30PW-M, TH cap, and SOT-23-3 footprints with 3D models
- Update connectors, power-reg, and mechanicals schematic sheets
- Rework PCB layout and update board STEP exports (r0 updated, r2 added)
- Regenerate interactive BOM

Co-Authored-By: Claude Fable 5 <noreply@anthropic.com>
Connections:
- net GPIO36 renamed enc-spi-copi
Changed lines of the file:
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@@
+		)
+	)
+	(global_label "enc-spi-copi"
+		(shape input)
+		(at 113.03 48.26 0)
+		(fields_autoplaced yes)
+		(effects
+			(font
+				(size 1.27 1.27)
+			)
+			(justify left)
+		)
+		(property "Intersheetrefs" "${INTERSHEET_REFS}"
+			(at 129.2595 48.26 0)
+			(hide yes)
+			(show_name no)
+			(do_not_autoplace no)
+			(effects
+				(font
+					(size 1.27 1.27)
+				)
+				(justify left)
+			)
 		)
 	)
@@
 			(hide yes)
 			(show_name no)
-			(do_not_autoplace no)
-			(effects
-				(font
-					(size 1.27 1.27)
-				)
-				(justify left)
-			)
-		)
-	)
-	(global_label "GPIO36"
-		(shape input)
-		(at 113.03 48.26 0)
-		(fields_autoplaced yes)
-		(effects
-			(font
-				(size 1.27 1.27)
-			)
-			(justify left)
-		)
-		(property "Intersheetrefs" "${INTERSHEET_REFS}"
-			(at 122.9095 48.26 0)
-			(hide yes)
-			(show_name no)

Commit message: Repo hygiene, CI as source of truth, and V1R2 design cleanup
Repository
- Sources only in pace-core/: untrack .history, lock files, .DS_Store,
  backups, layer PDFs, STEP exports, ibom. Regenerable outputs are
  gitignored; CI rebuilds them.
- Git LFS for Blender, PSD, video and curated renders (.gitattributes).
- Move brand artwork to graphics/, curated renders to docs/media/.
- Track the V1R2 fab package CSVs that the old gitignore hid.

CI
- KiBot builds gerbers, drill, fab zip, BOM (CSV/HTML with MPN and LCSC),
  position, ibom, IPC netlist, schematic and layer PDFs, DRC report,
  STEP and renders. REV is set from `git describe` on V*R* tags.
- ERC and DRC block PRs; tag builds publish a GitHub Release.
- README pin map is generated from the netlist (tools/gen_readme.py)
  and checked in CI.
- PR template with review checklist.

Design (ERC 0 errors, DRC 0 errors with schematic parity, netlist
connectivity verified identical across all 101 nets)
- Rename 49 nets to lowercase domain-kebab via tools/rename_nets.py.
- Add TITLE/PROJECT_CODE/REV/COMPANY text variables and title blocks on
  every sheet and the board.
- Net classes now carry both widths and colours: GND, 3V3, 5V, GND-USB,
  Batt, Motor-A/B/C. Remove High-Current-GND (its net never existed).
- Remove all 10 stale DRC exclusions; fold the shunt net-tie bridge copper
  into pad 2 and waive clearance around NT1..NT3 via pace-core.kicad_dru.
- Add Manufacturer/MPN/LCSC fields to every symbol and footprint.
- Fix capacitor symbols with input-typed pins, add PWR_FLAGs on GND and
  +BATT, convert duplicate local labels to global, complete the
  half-bridge bus alias, re-home symbols from missing libraries.

Docs
- docs/style-guide.md, decision records 0001-0003, errata, bring-up
  checklist. CLAUDE.md updated for the new layout and conventions.

Co-Authored-By: Claude Fable 5.1 <noreply@anthropic.com>
Parts:
- R11, R12, R13, R8, R9: symbol sparkfun_resistors:RESISTOR0603 -> specific-parts-lib:RESISTOR0603
Connections:
- net GPIO2 renamed mcu-io2
- net RX renamed uart-rx
- net TX renamed uart-tx
- net blue-ind renamed led-blue
- net boot renamed mcu-boot
- net green-ind renamed led-green
- net i2c-SCL renamed i2c-scl
- net i2c-SDA renamed i2c-sda
- net reset renamed mcu-reset
Other:
- note added: "Indicators & mcu-boot/rst"
- note removed: "Indicators & boot/rst"
- company: (none) -> ${COMPANY}
- title: (none) -> ${TITLE} - Sensing, Mechanicals, Config
