File: pace-core/pace-power-reg.kicad_sch (KiCad schematic)
At the start: 30 parts, among them U5 AMS1117-3.3, U6 XL7015E1, U7 REF35160QDBVR

Commit message: design checkpoint: v1 repackage — new connectors, footprints, and lay… (#1)
* design checkpoint: v1 repackage — new connectors, footprints, and layout updates

- Add JST SH/SR series, XT30PW-M, TH cap, and SOT-23-3 footprints with 3D models
- Update connectors, power-reg, and mechanicals schematic sheets
- Rework PCB layout and update board STEP exports (r0 updated, r2 added)
- Regenerate interactive BOM

Co-Authored-By: Claude Fable 5 <noreply@anthropic.com>

* update connectors schematic and PCB layout, refresh r2 STEP export

Co-Authored-By: Claude Fable 5 <noreply@anthropic.com>

* Repo hygiene, CI as source of truth, and V1R2 design cleanup

Repository
- Sources only in pace-core/: untrack .history, lock files, .DS_Store,
  backups, layer PDFs, STEP exports, ibom. Regenerable outputs are
  gitignored; CI rebuilds them.
- Git LFS for Blender, PSD, video and curated renders (.gitattributes).
- Move brand artwork to graphics/, curated renders to docs/media/.
- Track the V1R2 fab package CSVs that the old gitignore hid.

CI
- KiBot builds gerbers, drill, fab zip, BOM (CSV/HTML with MPN and LCSC),
  position, ibom, IPC netlist, schematic and layer PDFs, DRC report,
  STEP and renders. REV is set from `git describe` on V*R* tags.
- ERC and DRC block PRs; tag builds publish a GitHub Release.
- README pin map is generated from the netlist (tools/gen_readme.py)
  and checked in CI.
- PR template with review checklist.

Design (ERC 0 errors, DRC 0 errors with schematic parity, netlist
connectivity verified identical across all 101 nets)
- Rename 49 nets to lowercase domain-kebab via tools/rename_nets.py.
- Add TITLE/PROJECT_CODE/REV/COMPANY text variables and title blocks on
  every sheet and the board.
- Net classes now carry both widths and colours: GND, 3V3, 5V, GND-USB,
  Batt, Motor-A/B/C. Remove High-Current-GND (its net never existed).
- Remove all 10 stale DRC exclusions; fold the shunt net-tie bridge copper
  into pad 2 and waive clearance around NT1..NT3 via pa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
Parts:
- removed C22: 470uF 100V, specific-parts-lib:CAP-TH_BD16.0-P7.50-D1.2-FD, symbol specific-parts-lib:NXH100VB470M16*31.5LO
- removed TP26, TP27: TestPoint, TestPoint:TestPoint_Pad_D2.0mm, symbol Connector:TestPoint
- added C36, C37, C38, C39: PA100V22M6X9, specific-parts-lib:CAP-TH_BD6.3-P2.50-D0.6-FD, symbol specific-parts-lib:PA100V22M6X9
- C17: LCSC Part (none) -> C178585; LCSC part C178585 -> (none)
- D4: MPN (none) -> SS310
- U7: MPN (none) -> REF35160QDBVR; Manufacturer (none) -> Texas Instruments
Connections:
- net +BATT: now also C36.1, C37.1, C38.1, C39.1
- net GND: now also C36.2, C37.2, C38.2, C39.2
- net 1V6-REF renamed vref-1v6
Other:
- note added: "Al. Poly Size test"
- company: (none) -> ${COMPANY}
- title: (none) -> ${TITLE} - Power Regulation
- moved on the sheet: C19, C20, C21
