File: pace-core/pace-3-phase-inverter.kicad_sch (KiCad schematic)
At the start: 35 parts, among them J1 MotorOut, Q10 ISC0802NLSATMA1, Q11 ISC0802NLSATMA1, Q12 ISC0802NLSATMA1, Q7 ISC0802NLSATMA1, Q8 ISC0802NLSATMA1, Q9 ISC0802NLSATMA1, U2 DRV8353SRTAT

Commit message: Repo hygiene, CI as source of truth, and V1R2 design cleanup
Repository
- Sources only in pace-core/: untrack .history, lock files, .DS_Store,
  backups, layer PDFs, STEP exports, ibom. Regenerable outputs are
  gitignored; CI rebuilds them.
- Git LFS for Blender, PSD, video and curated renders (.gitattributes).
- Move brand artwork to graphics/, curated renders to docs/media/.
- Track the V1R2 fab package CSVs that the old gitignore hid.

CI
- KiBot builds gerbers, drill, fab zip, BOM (CSV/HTML with MPN and LCSC),
  position, ibom, IPC netlist, schematic and layer PDFs, DRC report,
  STEP and renders. REV is set from `git describe` on V*R* tags.
- ERC and DRC block PRs; tag builds publish a GitHub Release.
- README pin map is generated from the netlist (tools/gen_readme.py)
  and checked in CI.
- PR template with review checklist.

Design (ERC 0 errors, DRC 0 errors with schematic parity, netlist
connectivity verified identical across all 101 nets)
- Rename 49 nets to lowercase domain-kebab via tools/rename_nets.py.
- Add TITLE/PROJECT_CODE/REV/COMPANY text variables and title blocks on
  every sheet and the board.
- Net classes now carry both widths and colours: GND, 3V3, 5V, GND-USB,
  Batt, Motor-A/B/C. Remove High-Current-GND (its net never existed).
- Remove all 10 stale DRC exclusions; fold the shunt net-tie bridge copper
  into pad 2 and waive clearance around NT1..NT3 via pace-core.kicad_dru.
- Add Manufacturer/MPN/LCSC fields to every symbol and footprint.
- Fix capacitor symbols with input-typed pins, add PWR_FLAGs on GND and
  +BATT, convert duplicate local labels to global, complete the
  half-bridge bus alias, re-home symbols from missing libraries.

Docs
- docs/style-guide.md, decision records 0001-0003, errata, bring-up
  checklist. CLAUDE.md updated for the new layout and conventions.

Co-Authored-By: Claude Fable 5.1 <noreply@anthropic.com>
Parts:
- U2: symbol aaa-pace-project-specific:DRV8353SRTAT -> specific-parts-lib:DRV8353SRTAT
Connections:
- net 1V6-REF renamed vref-1v6
- net A-motor renamed mot-a
- net B-motor renamed mot-b
- net C-motor renamed mot-c
- net comm-spi-cipo renamed spi-cipo
- net comm-spi-clk renamed spi-clk
- net comm-spi-copi renamed spi-copi
- net gate-HA renamed gate-a-high
- net gate-HB renamed gate-b-high
- net gate-HC renamed gate-c-high
- net gate-LA renamed gate-a-low
- net gate-LB renamed gate-b-low
- net gate-LC renamed gate-c-low
- net motor-fault renamed drv-fault
- net pwm.A-high renamed pwm.pwm-a-high
- net pwm.A-low renamed pwm.pwm-a-low
- net pwm.B-high renamed pwm.pwm-b-high
- net pwm.B-low renamed pwm.pwm-b-low
- net pwm.C-high renamed pwm.pwm-c-high
- net pwm.C-low renamed pwm.pwm-c-low
- net pwm.MC-enable renamed pwm.drv-enable
- net shunts.A-isense renamed shunts.isense-a
- net shunts.B-isense renamed shunts.isense-b
- net shunts.C-isense renamed shunts.isense-c
- net src-NA renamed shunt-a-n
- net src-NB renamed shunt-b-n
- net src-NC renamed shunt-c-n
- net src-PA renamed shunt-a-p
- net src-PB renamed shunt-b-p
- net src-PC renamed shunt-c-p
Other:
- company: (none) -> ${COMPANY}
- title: (none) -> ${TITLE} - Gate Driver and Half Bridges
