File: pace-core/pace-connectors-sheet.kicad_sch (KiCad schematic)
At the start: 29 parts, among them CN1 XT60PW-M, J2 Wiz5500-Coprocessor-BoB, SW3 DPDT, U12 SM06B-SRSS-TB, U13 SM06B-SRSS-TB, U3 USBLC6-2P6, U4 ADUM3160BRWZ-RL

Commit message: ci: use erc/drc preflights, single KiBot step, PWR_FLAG on +5V
- KiBot 1.9 rejected `warnings_as_errors` on the legacy run_drc preflight;
  switch to the `erc` and `drc` preflights with HTML+JSON reports.
- Collapse the two KiBot steps into one: the first step's `skip: all`
  skipped the checks it was meant to run.
- KiCad 10.0.5 in the CI image flags +5V as undriven (the buck output pin
  is Unspecified); add a PWR_FLAG. Merge C17's duplicate "LCSC part" field.
- Document the local Docker run and the two source files KiBot rewrites.

Validated locally with ghcr.io/inti-cmnb/kicad10_auto_full: ERC 0 errors,
DRC 0 errors, all 12 outputs produced, README check passes.

Co-Authored-By: Claude Fable 5.1 <noreply@anthropic.com>
Changed lines of the file:
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@@
+		)
+	)
+	(symbol
+		(lib_id "power:PWR_FLAG")
+		(at 34.29 190.5 0)
+		(unit 1)
+		(body_style 1)
+		(exclude_from_sim no)
+		(in_bom yes)
+		(on_board yes)
+		(in_pos_files yes)
+		(dnp no)
+		(fields_autoplaced yes)
+		(property "Reference" "#FLG012"
+			(at 34.29 188.595 0)
+			(hide yes)
+			(show_name no)
+			(do_not_autoplace no)
+			(effects
+				(font
+					(size 1.27 1.27)
+				)
+			)
+		)
+		(property "Value" "PWR_FLAG"
+			(at 34.29 186.69 0)
+			(show_name no)
+			(do_not_autoplace no)
+			(effects
+				(font
+					(size 1.27 1.27)
+				)
+			)
+		)
+		(property "Footprint" ""
+			(at 34.29 190.5 0)
+			(hide yes)
+			(show_name no)
+			(do_not_autoplace no)
+			(effects
+				(font
+					(size 1.27 1.27)
+				)
+			)
+		)
+		(property "Datasheet" ""
+			(at 34.29 190.5 0)
+			(hide yes)
+			(show_name no)
+			(do_not_autoplace no)
+			(effects
+				(font
+					(size 1.27 1.27)
+				)
+			)
+		)
+		(property "Description" "Special symbol for telling ERC where power comes from"
+			(at 34.29 190.5 0)
+			(hide yes)
+			(show_name no)
+			(do_not_autoplace no)
+			(effects
+				(font
+					(size 1.27 1.27)
+				)
+			)
+		)
+		(pin "1"
+		)
+		(instances
+			(project "pace-core"
+				(path "/a993745c-3062-41b3-ae55-cf32fb6be737/f6e8a3c1-3318-4f1a-a32b-34eb1543d997"
+					(reference "#FLG012")
+					(unit 1)
+				)
+			)
 		)
 	)
