File: pace-core/pace-connectors-sheet.kicad_sch (KiCad schematic)
At the start: 22 parts, among them CN1 XT90PW-M.G.Y, J2 Wiz5500-Coprocessor-BoB, J3 Conn_01x05, J6 Conn_01x05, SW3 DPDT, U3 USBLC6-2P6, U4 ADUM3160BRWZ-RL

Commit message: design checkpoint: v1 repackage — new connectors, footprints, and lay… (#1)
* design checkpoint: v1 repackage — new connectors, footprints, and layout updates

- Add JST SH/SR series, XT30PW-M, TH cap, and SOT-23-3 footprints with 3D models
- Update connectors, power-reg, and mechanicals schematic sheets
- Rework PCB layout and update board STEP exports (r0 updated, r2 added)
- Regenerate interactive BOM

Co-Authored-By: Claude Fable 5 <noreply@anthropic.com>

* update connectors schematic and PCB layout, refresh r2 STEP export

Co-Authored-By: Claude Fable 5 <noreply@anthropic.com>

* Repo hygiene, CI as source of truth, and V1R2 design cleanup

Repository
- Sources only in pace-core/: untrack .history, lock files, .DS_Store,
  backups, layer PDFs, STEP exports, ibom. Regenerable outputs are
  gitignored; CI rebuilds them.
- Git LFS for Blender, PSD, video and curated renders (.gitattributes).
- Move brand artwork to graphics/, curated renders to docs/media/.
- Track the V1R2 fab package CSVs that the old gitignore hid.

CI
- KiBot builds gerbers, drill, fab zip, BOM (CSV/HTML with MPN and LCSC),
  position, ibom, IPC netlist, schematic and layer PDFs, DRC report,
  STEP and renders. REV is set from `git describe` on V*R* tags.
- ERC and DRC block PRs; tag builds publish a GitHub Release.
- README pin map is generated from the netlist (tools/gen_readme.py)
  and checked in CI.
- PR template with review checklist.

Design (ERC 0 errors, DRC 0 errors with schematic parity, netlist
connectivity verified identical across all 101 nets)
- Rename 49 nets to lowercase domain-kebab via tools/rename_nets.py.
- Add TITLE/PROJECT_CODE/REV/COMPANY text variables and title blocks on
  every sheet and the board.
- Net classes now carry both widths and colours: GND, 3V3, 5V, GND-USB,
  Batt, Motor-A/B/C. Remove High-Current-GND (its net never existed).
- Remove all 10 stale DRC exclusions; fold the shunt net-tie bridge copper
  into pad 2 and waive clearance around NT1..NT3 via pa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
Parts:
- removed CN1: XT90PW-M.G.Y, specific-parts-lib:CONN-TH_XT90PW-M.G.Y, symbol specific-parts-lib:XT90PW-M.G.Y
- removed J3, J6: Conn_01x05, Connector_JST:JST_XA_B05B-XASK-1-A_1x05_P2.50mm_Vertical, symbol Connector_Generic:Conn_01x05
- added C40, C41, C42: 1nF, Capacitor_SMD:C_0402_1005Metric, symbol Device:C_Small
- added CN1: XT60PW-M, specific-parts-lib:CONN-TH_XT60PW-M, symbol specific-parts-lib:XT60PW-M
- added JP5: SolderJumper_3_Bridged12, Jumper:SolderJumper-3_P1.3mm_Open_RoundedPad1.0x1.5mm, symbol Jumper:SolderJumper_3_Open
- added R25, R33, R34: 100R, Resistor_SMD:R_0402_1005Metric, symbol Device:R_Small_US
- added U12, U13: SM06B-SRSS-TB, specific-parts-lib:CONN-SMD_SM06B-SRSS-TB-LF-SN, symbol specific-parts-lib:SM06B-SRSS-TB
- R4, R5, R6, R7: symbol sparkfun_resistors:RESISTOR0603 -> specific-parts-lib:RESISTOR0603
- U3: MPN (none) -> USBLC6-2P6; Manufacturer (none) -> STMicroelectronics
Connections:
- net +3V3: now also JP4.1 (A), JP5.1 (A), U12.5; no longer JP4.3 (B)
- net +5V: now also JP4.3 (B), JP5.3 (B); no longer JP4.1 (A)
- net +BATT: now also CN1.2 (+)
- net GND: now also C40.2, C41.2, C42.2, U12.6, U13.6
- net GNDPWR: now also CN1.1 (-), CN1.3, CN1.4
- net enc-spi-cipo: now also U12.4
- net enc-spi-clk: now also U12.3
- net enc-spi-cs: now also U12.1
- net at R7.1: now also U4.6 (UD–); no longer U4.7 (UD+)
- net at R6.1: now also U4.7 (UD+); no longer U4.6 (UD–)
- net hall-vpull: now reaches R18.2, R19.2, R20.2
- net hall-vpull: now also JP5.2 (C); no longer JP4.2 (C)
- net A-halls: no longer names the net of R20.1
- net A-halls: now also R34.2, U13.4
- net B-Halls: no longer names the net of R19.1
- net B-Halls: now also R33.2, U13.3
- net C-Halls: no longer names the net of R18.1
- net C-Halls: now also R25.2, U13.2
- net comm-irq renamed eth-irq
- net comm-reset renamed eth-reset
- net comm-spi-cipo renamed spi-cipo
- net comm-spi-clk renamed spi-clk
- net comm-spi-copi renamed spi-copi
- net comm-spi-cs renamed eth-spi-cs
- net usb_d+ renamed usb-dp
- net usb_d- renamed usb-dm
- new net enc-spi-copi: U12.2
- new net hall-a: C42.1, R34.1
- new net hall-b: C41.1, R33.1
- new net hall-c: C40.1, R25.1
- new net hall-vcc: JP4.2 (C), U13.5
- no-connect marks 5 -> 10
Other:
- note added: "SPI Encoder Connector"
- note removed: "MT6701 Encoder Connector"
- company: (none) -> ${COMPANY}
- title: (none) -> ${TITLE} - Connectors
- moved on the sheet: J2, R18, R19, R20, R23, R24, SW3
