File: pr-previews/1/44d78f0/pace-core.kicad_pcb (KiCad board)
At the start: 4 copper layers, 100 x 80.1 mm, 173 parts, among them CN1 XT60PW-M, CN2 SMTSOM330BTR, CN3 SMTSOM330BTR, CN4 SMTSOM330BTR, CN5 SMTSOM330BTR, CN6 SMTSOM330BTR, CN7 SMTSOM330BTR, J1 MotorOut, J2 Wiz5500-Coprocessor-BoB, J4 Conn_02x05_Odd_Even, Q10 ISC0802NLSATMA1, Q11 ISC0802NLSATMA1, Q12 ISC0802NLSATMA1, Q7 ISC0802NLSATMA1, Q8 ISC0802NLSATMA1, Q9 ISC0802NLSATMA1, SW1 SKRPACE010, SW2 SKRPACE010, SW3 DPDT, U1 ESP32-S3-WROOM-1, U10 LM75ADP,118, U11 LM75ADP,118, U12 SM06B-SRSS-TB, U13 SM06B-SRSS-TB, U2 DRV8353SRTAT, U3 USBLC6-2P6, U4 ADUM3160BRWZ-RL, U5 AMS1117-3.3, U6 XL7015E1, U7 REF35160QDBVR, U8 LM75ADP,118, U9 LM75ADP,118

Commit message: Update Kiri output for PR #1
Parts:
- added kibuzzard-6A7D445B: G***, kibuzzard-6A7D445B, F.Cu at (186.7, 127.2)
- added kibuzzard-6A7D4481: G***, kibuzzard-6A7D4481, F.Cu at (189.3, 126.3)
- moved kibuzzard-6A76AD71 18.4 mm to (184.1, 123.6), turned to 0 degrees
- moved kibuzzard-6A76AD5A 15.1 mm to (184.0, 121.0), turned to 0 degrees
- moved kibuzzard-6A76A991 2.83 mm to (193.8, 101.4)
- moved kibuzzard-6A76A9E7 2.65 mm to (191.1, 101.8)
- moved kibuzzard-6A79703A 1.22 mm to (192.1, 117.1)
- moved kibuzzard-6A797050 1.10 mm to (192.1, 106.0)
Connections:
- net /A-high renamed /pwm-a-high
- net /A-isense renamed /isense-a
- net /A-low renamed /pwm-a-low
- net /B-high renamed /pwm-b-high
- net /B-isense renamed /isense-b
- net /B-low renamed /pwm-b-low
- net /C-high renamed /pwm-c-high
- net /C-isense renamed /isense-c
- net /C-low renamed /pwm-c-low
- net /Connectors/v_halls_pwr renamed /Connectors/hall-vcc
- net /Connectors/v_pullup renamed /Connectors/hall-vpull
- net /Gate Driver and Half Bridges/gate-HA renamed /Gate Driver and Half Bridges/gate-a-high
- net /Gate Driver and Half Bridges/gate-HB renamed /Gate Driver and Half Bridges/gate-b-high
- net /Gate Driver and Half Bridges/gate-HC renamed /Gate Driver and Half Bridges/gate-c-high
- net /Gate Driver and Half Bridges/gate-LA renamed /Gate Driver and Half Bridges/gate-a-low
- net /Gate Driver and Half Bridges/gate-LB renamed /Gate Driver and Half Bridges/gate-b-low
- net /Gate Driver and Half Bridges/gate-LC renamed /Gate Driver and Half Bridges/gate-c-low
- net /Gate Driver and Half Bridges/src-NA renamed /Gate Driver and Half Bridges/shunt-a-n
- net /Gate Driver and Half Bridges/src-NB renamed /Gate Driver and Half Bridges/shunt-b-n
- net /Gate Driver and Half Bridges/src-NC renamed /Gate Driver and Half Bridges/shunt-c-n
- net /Gate Driver and Half Bridges/src-PA renamed /Gate Driver and Half Bridges/shunt-a-p
- net /Gate Driver and Half Bridges/src-PB renamed /Gate Driver and Half Bridges/shunt-b-p
- net /Gate Driver and Half Bridges/src-PC renamed /Gate Driver and Half Bridges/shunt-c-p
- net /MC-enable renamed /drv-enable
- net 1V6-REF renamed vref-1v6
- net A-halls renamed hall-a
- net A-motor renamed mot-a
- net B-Halls renamed hall-b
- net B-motor renamed mot-b
- net C-Halls renamed hall-c
- net C-motor renamed mot-c
- net GPIO2 renamed mcu-io2
- net RX renamed uart-rx
- net TX renamed uart-tx
- net blue-ind renamed led-blue
- net boot renamed mcu-boot
- net comm-irq renamed eth-irq
- net comm-reset renamed eth-reset
- net comm-spi-cipo renamed spi-cipo
- net comm-spi-clk renamed spi-clk
- net comm-spi-copi renamed spi-copi
- net comm-spi-cs renamed eth-spi-cs
- net green-ind renamed led-green
- net i2c-SCL renamed i2c-scl
- net i2c-SDA renamed i2c-sda
- net motor-fault renamed drv-fault
- net reset renamed mcu-reset
- net usb_d+ renamed usb-dp
- net usb_d- renamed usb-dm
Routing:
- net +3V3: track 322.9 -> 316.8 mm
- net /Connectors/hall-vpull: track 27.7 -> 23.4 mm
- net GND: vias 460 -> 437
